File: ME433Schematic.sch (EAGLE design)
At the start: 11 parts

Commit message: need to know if power plane is good idea re capacitors
Parts:
- removed U$10: 10UF, ME433Library:10UF
- removed U$11, U$5: 0.1UF, ME433Library:0.1UF
- removed U$4: 8MHZRESONATOR, ME433Library:8MHZRESONATOR
- removed U$6: GREENLED, ME433Library:GREENLED
- removed U$7, U$9: 330OHM, ME433Library:330OHM
- added C1, C2: 10uF, ME433Library:CPOL-USB45181B
- added C3, C4, C5, C6: 0.1uF, ME433Library:C-US025-025X050
- added C7: 0.1uF, ME433Library:C-US025-030X050
- added J1: (no value), ME433Library:M06SILK_FEMALE_PTH
- added J2, J3: (no value), ME433Library:M08
- added LED1: RED, ME433Library:LED3MM
- added LED2: GREEN, ME433Library:LED3MM
- added R1, R3: 10K, ME433Library:R-US_0207/10
- added R2, R4: 330, ME433Library:R-US_0207/10
- added U$12: USBMINIB, ME433Library:USBMINIB
- added U$13: MCP1702TO, ME433Library:MCP1702TO
- added U$18: SLIDESWITCH, ME433Library:SLIDESWITCH
- U$2: value 330OHM -> 8MHZRESONATOR; device ME433Library:330OHM -> ME433Library:8MHZRESONATOR
Connections:
- removed net N$4: U$1.11.SOSCI/RPB4/RB4, U$8.1.IN, U$9.2
- removed net N$5: U$1.12.SOSCO/RPA4/T1CK/CTED9/PMA1/RA4, U$6.1.+
- removed net N$8: U$1.23.VUSB3V3, U$11.1
- new net +5V: C6.1, J3.2, U$1.15.VBUS, U$13.2.VIN, U$18.1.OUT
- new net A0: J2.8, U$1.2.PGED3/VREF+/CVREF+/AN0/C3INC/RPA0/CTED1/PMD7/RA0
- new net A1: J2.7, U$1.3.PGEC3/VREF-/CVREF-/AN1/RPA1/CTED2/PMD6/RA1
- new net A4: J2.3, LED2.1.+, U$1.12.SOSCO/RPA4/T1CK/CTED9/PMA1/RA4
- new net B13: J3.6, U$1.24.AN11/RPB13/CTPLS/PMRD/RB13
- new net B14: J3.7, U$1.25.CVREFOUT/AN10/C3INB/RPB14/SCK1/CTED5/PMWR/RB14
- new net B15: J3.8, U$1.26.AN9/C3INA/RPB15/SCK2/CTED6/PMCS1/RB15
- new net B2: J2.6, U$1.6.AN4/C1INB/C2IND/RPB2/SDA2/CTED13/RB2
- new net B3: J2.5, U$1.7.AN5/C1INA/C2INC/RTCC/RPB3/SCL2/RB3
- new net B4: J2.4, R3.2, U$1.11.SOSCI/RPB4/RB4, U$8.1.IN
- new net B7: J3.3, U$1.16.TDI/RPB7/CTED3/PMD5/INT0/RB7
- new net B8: J3.4, U$1.17.TCK/RPB8/SCL1/CTED10/PMD4/RB8
- new net B9: J3.5, U$1.18.TDO/RPB9/SDA1/CTED4/PMD3/RB9
- new net D+: U$1.21.PGED2/RPB10/CTED11/PMD2/RB10, U$12.3.D+
- new net D-: U$1.22.PGEC2/TMS/RPB11/PMD1/RB11, U$12.2.D-
- new net ID: U$1.14.TMS/RPB5/USBID/RB5, U$12.4.ID
- new net MCLR: J1.1, R1.2, U$1.1.MCLR, U$3.1.IN
- new net N$11: LED1.2.-, R2.2
- new net PEGC1: J1.5, U$1.5.PGEC1/AN3/C1INC/C2INA/RPB1/CTED12/PMD1/RB1
- new net PEGD1: J1.4, U$1.4.PGED1/AN2/C1IND/C2INB/C3IND/RPB0/PMD0/RB0
- net +3V3: now also C1.+, C3.1, C4.1, C5.1, C7.1, J1.2, J2.2, LED1.1.+, R1.1, R3.1, U$1.23.VUSB3V3, U$1.28.AVDD, U$13.VOU3.T; no longer U$2.1, U$5.1, U$9.1
- net GND: now also C1.-, C2.-, C3.2, C4.2, C5.2, C6.2, C7.2, J1.3, J2.1, J3.1, R2.1, R4.1, U$1.27.AVSS, U$12.5.GND, U$13.1.GND, U$2.2.GND; no longer U$10.-, U$11.2, U$4.3.GND, U$5.2, U$7.2
- net N$1: now also U$12.1.VBUS, U$18.3.COMMON; no longer U$1.1.MCLR, U$2.2, U$3.1.IN
- net N$2: now also U$2.3.OSC2; no longer U$4.2.OSC2
- net N$3: now also U$2.1.OSC1; no longer U$4.1.OSC1
- net N$6: now also C2.+; no longer U$10.+
- net N$7: now also LED2.2.-, R4.2; no longer U$6.2.-, U$7.1

Commit message: Ready to be checked before order, looked good on Seeed, holes were off by 10x-100x in Mayhew labs
Parts:
- removed C7: 0.1uF, ME433Library:C-US025-030X050
- U$3: value PUSHSWITCH -> MCLR
Connections:
- net +3V3: no longer C7.1
- net GND: no longer C7.2
Changed lines of the file:
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@@
 <part name="+3V1" library="ME433Library" deviceset="+3V3" device=""/>
 <part name="GND1" library="ME433Library" deviceset="GND" device=""/>
-<part name="U$3" library="ME433Library" deviceset="PUSHSWITCH" device=""/>
+<part name="U$3" library="ME433Library" deviceset="PUSHSWITCH" device="" value="MCLR"/>
 <part name="GND2" library="ME433Library" deviceset="GND" device=""/>
 <part name="GND3" library="ME433Library" deviceset="GND" device=""/>
@@
 <part name="GND12" library="ME433Library" deviceset="GND" device=""/>
 <part name="P+3" library="ME433Library" deviceset="+5V" device=""/>
-<part name="C7" library="ME433Library" deviceset="C-US" device="025-030X050" value="0.1uF"/>
 <part name="GND14" library="ME433Library" deviceset="GND" device=""/>
 <part name="+3V8" library="ME433Library" deviceset="+3V3" device=""/>
@@
 <instance part="GND12" gate="1" x="99.06" y="-10.16" rot="R270"/>
 <instance part="P+3" gate="1" x="149.86" y="33.02" rot="R270"/>
-<instance part="C7" gate="G$1" x="154.94" y="66.04"/>
 <instance part="GND14" gate="1" x="167.64" y="60.96" rot="R90"/>
 <instance part="+3V8" gate="G$1" x="167.64" y="73.66"/>
@@
 <wire x1="142.24" y1="66.04" x2="149.86" y2="66.04" width="0.1524" layer="91"/>
 <wire x1="149.86" y1="66.04" x2="149.86" y2="68.58" width="0.1524" layer="91"/>
-<pinref part="C7" gate="G$1" pin="1"/>
-<wire x1="149.86" y1="68.58" x2="154.94" y2="68.58" width="0.1524" layer="91"/>
 <pinref part="+3V8" gate="G$1" pin="+3V3"/>
-<wire x1="154.94" y1="68.58" x2="167.64" y2="68.58" width="0.1524" layer="91"/>
+<wire x1="149.86" y1="68.58" x2="167.64" y2="68.58" width="0.1524" layer="91"/>
 <wire x1="167.64" y1="68.58" x2="167.64" y2="71.12" width="0.1524" layer="91"/>
-<junction x="154.94" y="68.58"/>
 </segment>
 </net>
@@
 <wire x1="142.24" y1="63.5" x2="152.4" y2="63.5" width="0.1524" layer="91"/>
 <wire x1="152.4" y1="63.5" x2="152.4" y2="60.96" width="0.1524" layer="91"/>
-<pinref part="C7" gate="G$1" pin="2"/>
-<wire x1="152.4" y1="60.96" x2="154.94" y2="60.96" width="0.1524" layer="91"/>
 <pinref part="GND14" gate="1" pin="GND"/>
-<wire x1="154.94" y1="60.96" x2="165.1" y2="60.96" width="0.1524" layer="91"/>
-<junction x="154.94" y="60.96"/>
+<wire x1="152.4" y1="60.96" x2="165.1" y2="60.96" width="0.1524" layer="91"/>
 </segment>
 </net>
