File: ME433Schematic.brd (EAGLE design)
At the start: 50 x 50 mm, 23 parts

Commit message: Ready to be checked before order, looked good on Seeed, holes were off by 10x-100x in Mayhew labs
Parts:
- removed C7: 0.1uF, ME433Library:C025-030X050
- U$3: value PUSHSWITCH -> MCLR
- moved C3 58.7 mm to (24.1, 4.76), turned to 180 degrees
- moved C1 40.9 mm to (27.3, 45.4)
- moved C5 38.2 mm to (32.1, 27.9)
- moved C4 20.3 mm to (31.1, 39.4), turned to 270 degrees
- moved U$12 2.62 mm to (39.7, 46.7)
- moved U$18 2.56 mm to (48.3, 42.5)
- moved C6 2.25 mm to (43.5, 37.8)
- moved U$13 2.22 mm to (31.4, 47.0)
- moved U$3 1.71 mm to (2.86, 40.6)
Connections:
- net +3V3: no longer C7.1
- net GND: no longer C7.2
Routing:
- net +5V: track 77.4 -> 67.6 mm
- net ID: track 52.3 -> 58.1 mm, vias 1 -> 3
- net N$7: track 0.00 -> 2.54 mm
- net D-: track 30.8 -> 33.3 mm, vias 2 -> 1
- net D+: track 27.3 -> 29.7 mm
Other:
- board text added: "Aidan Jenkins ME433 Spring 2016"
- board text added: "MCLR"
- board text added: "USER"

Commit message: Board updated ready to review
Routing:
- net ID: track 58.1 -> 53.2 mm
Other:
- board text added: "3.3V"
- board text added: "5V"
- board text added: "GND"
Changed lines of the file:
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@@
+<vertex x="18.0975" y="46.6725"/>
+</polygon>
+<text x="2.54" y="19.685" size="1.778" layer="22" rot="MR180">3.3V</text>
+<text x="7.3025" y="15.5575" size="1.778" layer="22" rot="MR0">GND</text>
+<text x="49.2125" y="13.0175" size="1.778" layer="22" rot="MR0">GND</text>
+<text x="44.45" y="13.0175" size="1.778" layer="21">GND</text>
+<text x="44.45" y="16.51" size="1.778" layer="21">5V</text>
+<text x="46.99" y="16.51" size="1.778" layer="22" rot="MR0">5V</text>
+<text x="0.3175" y="13.335" size="1.778" layer="21">GND</text>
+<text x="2.8575" y="18.0975" size="1.778" layer="21">3.3V</text>
+<polygon width="0.4064" layer="21">
+<vertex x="16.8275" y="47.9425"/>
+<vertex x="18.0975" y="49.2125"/>
+<vertex x="18.0975" y="46.99"/>
+<vertex x="18.0975" y="46.6725"/>
+</polygon>
+<polygon width="0.4064" layer="22">
+<vertex x="16.8275" y="47.9425"/>
+<vertex x="18.0975" y="49.2125"/>
 <vertex x="18.0975" y="46.6725"/>
 </polygon>
@@
 <element name="R2" library="ME433Library" package="0207/10" value="330" x="16.51" y="45.085"/>
 <element name="R3" library="ME433Library" package="0207/10" value="10K" x="6.35" y="19.05" smashed="yes" rot="R90">
-<attribute name="VALUE" x="6.985" y="16.7894" size="1.27" layer="27" ratio="10" rot="R90"/>
+<attribute name="VALUE" x="8.89" y="15.5194" size="1.27" layer="27" ratio="10" rot="R90"/>
 </element>
 <element name="R4" library="ME433Library" package="0207/10" value="330" x="8.255" y="3.175" smashed="yes">
@@
 <contactref element="U$1" pad="23"/>
 <contactref element="C4" pad="1"/>
-<polygon width="0.4064" layer="1">
+<polygon width="0.4064" layer="1" isolate="0.3048">
 <vertex x="-5.08" y="-2.54"/>
 <vertex x="-5.08" y="58.42"/>
@@
 <contactref element="J3" pad="1"/>
 <contactref element="J2" pad="1"/>
-<polygon width="0.4064" layer="16">
+<polygon width="0.4064" layer="16" isolate="0.3048">
 <vertex x="-5.08" y="-2.54"/>
 <vertex x="-5.08" y="55.88"/>
@@
 <wire x1="38.4175" y1="43.18" x2="36.5125" y2="43.18" width="0.4064" layer="16"/>
 <wire x1="36.5125" y1="43.18" x2="35.56" y2="42.2275" width="0.4064" layer="16"/>
-<wire x1="35.56" y1="42.2275" x2="35.56" y2="40.005" width="0.4064" layer="16"/>
-<wire x1="35.56" y1="40.005" x2="35.8775" y2="39.6875" width="0.4064" layer="16"/>
-<wire x1="35.8775" y1="39.6875" x2="37.1475" y2="39.6875" width="0.4064" layer="16"/>
-<wire x1="37.1475" y1="39.6875" x2="38.1" y2="38.735" width="0.4064" layer="16"/>
-<wire x1="38.1" y1="38.735" x2="38.1" y2="34.29" width="0.4064" layer="16"/>
-<via x="38.1" y="34.29" extent="1-16" drill="0.6"/>
-<wire x1="38.1" y1="34.29" x2="24.13" y2="34.29" width="0.4064" layer="1"/>
+<via x="34.6075" y="34.29" extent="1-16" drill="0.6"/>
+<wire x1="34.6075" y1="34.29" x2="24.13" y2="34.29" width="0.4064" layer="1"/>
 <via x="24.13" y="34.29" extent="1-16" drill="0.6"/>
 <wire x1="24.13" y1="34.29" x2="24.13" y2="7.62" width="0.4064" layer="16"/>
 <via x="24.13" y="7.62" extent="1-16" drill="0.6"/>
 <wire x1="24.13" y1="7.62" x2="20.32" y2="7.62" width="0.4064" layer="1"/>
+<wire x1="35.56" y1="42.2275" x2="35.56" y2="35.2425" width="0.4064" layer="16"/>
+<wire x1="35.56" y1="35.2425" x2="34.6075" y2="34.29" width="0.4064" layer="16"/>
 </signal>
 <signal name="+5V">
